Commit message: Bumper publishing

File: create_description/urdf/create_base.urdf.xacro (robot description, xacro)
@@ -66,4 +66,10 @@
     </link>
     <link name="wall_sensor_link">
+    <collision name="wall_sensor_collision">
+      <origin xyz="0 0 0" rpy="0 0 0"/>
+      <geometry>
+        <box size="0.2 0.1 0.2"/>
+      </geometry>
+    </collision>
     <inertial>
       <mass value="0.01" />

File: create_description/urdf/create_base_gazebo.urdf.xacro (robot description, xacro)
@@ -78,24 +78,18 @@
   <xacro:macro name="sim_create_wall_sensor">
     <gazebo reference="wall_sensor_link">
-      <sensor type="ray" name="wall_sensor">
+      <sensor type="contact" name="wall_sensor">
         <always_on>true</always_on>
-        <update_rate>20.0</update_rate>
-        <pose>0 0 0 0 0 0</pose>
-        <visualize>false</visualize>
-        <ray>
-          <scan>
-            <horizontal>
-              <samples>1</samples>
-              <resolution>1</resolution>
-              <min_angle>0</min_angle>
-              <max_angle>0</max_angle>
-            </horizontal>
-          </scan>
-          <range>
-            <min>0.0160</min>
-            <max>0.04</max>
-            <resolution>0.1</resolution>
-          </range>
-        </ray>
+        <update_rate>10.0</update_rate>
+        <visualize>true</visualize>
+        <contact>
+          <collision>base_footprint_fixed_joint_lump__wall_sensor_collision_collision_2</collision>
+        </contact>
+        <plugin name="gazebo_ros_bumper_controller" filename="libgazebo_ros_bumper.so">
+            <bumperTopicName>wall_sensor_bumper</bumperTopicName>
+            <!-- <frameName>wall_sensor_link</frameName> -->
+            <!-- <contact>
+              <collision>wall_sensor_collision</collision>
+            </contact> -->
+        </plugin>
       </sensor>
     </gazebo>

Commit message: Bumper contact sensor

File: create_description/urdf/create_base.urdf.xacro (robot description, xacro)
@@ -199,4 +199,5 @@
     <!-- Simulation sensors -->
     <xacro:sim_create_base/>
+    <xacro:sim_create_bump_sensor/>
     <xacro:sim_create_wall_sensor/>
     <xacro:sim_create_cliff_sensors/>

File: create_description/urdf/create_base_gazebo.urdf.xacro (robot description, xacro)
@@ -76,4 +76,21 @@
     </gazebo>
   </xacro:macro>
+  <xacro:macro name="sim_create_bump_sensor">
+    <gazebo reference="base_link">
+      <sensor name="bumper" type="contact">
+        <always_on>true</always_on>
+        <update_rate>20.0</update_rate>
+        <maxContacts>10</maxContacts>
+        <pose>0 0 0 0 0 0</pose>
+        <visualize>false</visualize>
+        <contact>
+          <collision>base_footprint_fixed_joint_lump__base_link_collision_1</collision>
+        </contact>
+        <plugin name="gazebo_ros_bumper_controller" filename="libgazebo_ros_bumper.so">
+          <bumperTopicName>/sim/bumper</bumperTopicName>
+        </plugin>
+      </sensor>
+    </gazebo>
+  </xacro:macro>
   <xacro:macro name="sim_create_wall_sensor">
     <gazebo reference="wall_sensor_link">

Commit message: Fix Gazebo invalid inertia error for base_footprint link
Co-authored-by: nnarain <8395093+nnarain@users.noreply.github.com>
Agent-Logs-Url: https://github.com/nnarain/create_robot/sessions/801049ef-934e-4c54-8e51-f3dc7b0d1717

File: create_description/urdf/create_base.urdf.xacro (robot description, xacro)
@@ -32,4 +32,9 @@
     <xacro:include filename="$(find create_description)/urdf/create_base_gazebo.urdf.xacro" />
     <link name="base_footprint">
+    <inertial>
+      <origin xyz="0 0 0" />
+      <mass value="0.001" />
+      <inertia ixx="0.0001" ixy="0.0" ixz="0.0" iyy="0.0001" iyz="0.0" izz="0.0001" />
+    </inertial>
     <visual>
       <origin xyz="0 0 0" rpy="0 0 0" />
