Commit message: Light sensor URDF for Create 2

File: create_description/urdf/create_2.urdf.xacro (robot description, xacro)
@@ -6,3 +6,78 @@
     <mesh filename="package://create_description/meshes/create_2.dae" />
   </xacro:create_base>
+  <!-- Bumper Light Sensors -->
+  <link name="left_light_sensor_link">
+  <inertial>
+    <mass value="0.01" />
+    <origin xyz="0 0 0" />
+    <inertia ixx="0.001" ixy="0.0" ixz="0.0" iyy="0.001" iyz="0.0" izz="0.001" />
+  </inertial>
+  </link>
+  <link name="left_front_light_sensor_link">
+  <inertial>
+    <mass value="0.01" />
+    <origin xyz="0 0 0" />
+    <inertia ixx="0.001" ixy="0.0" ixz="0.0" iyy="0.001" iyz="0.0" izz="0.001" />
+  </inertial>
+  </link>
+  <link name="left_center_light_sensor_link">
+  <inertial>
+    <mass value="0.01" />
+    <origin xyz="0 0 0" />
+    <inertia ixx="0.001" ixy="0.0" ixz="0.0" iyy="0.001" iyz="0.0" izz="0.001" />
+  </inertial>
+  </link>
+  <link name="right_light_sensor_link">
+  <inertial>
+    <mass value="0.01" />
+    <origin xyz="0 0 0" />
+    <inertia ixx="0.001" ixy="0.0" ixz="0.0" iyy="0.001" iyz="0.0" izz="0.001" />
+  </inertial>
+  </link>
+  <link name="right_front_light_sensor_link">
+  <inertial>
+    <mass value="0.01" />
+    <origin xyz="0 0 0" />
+    <inertia ixx="0.001" ixy="0.0" ixz="0.0" iyy="0.001" iyz="0.0" izz="0.001" />
+  </inertial>
+  </link>
+  <link name="right_center_light_sensor_link">
+  <inertial>
+    <mass value="0.01" />
+    <origin xyz="0 0 0" />
+    <inertia ixx="0.001" ixy="0.0" ixz="0.0" iyy="0.001" iyz="0.0" izz="0.001" />
+  </inertial>
+  </link>
+  <joint name="base_left_light_sensor_joint" type="fixed">
+    <origin xyz="0.02469 0.1580 0.042" rpy="0 0 1.4158" />
+    <parent link="base_link" />
+    <child link="left_light_sensor_link" />
+  </joint>
+  <joint name="base_left_front_light_sensor_joint" type="fixed">
+    <origin xyz="0.0938 0.12957 0.042" rpy="0 0 0.9438" />
+    <parent link="base_link" />
+    <child link="left_front_light_sensor_link" />
+  </joint>
+  <joint name="base_left_center_light_sensor_joint" type="fixed">
+    <origin xyz="0.1425 0.07273 0.042" rpy="0 0 0.4719" />
+    <parent link="base_link" />
+    <child link="left_center_light_sensor_link" />
+  </joint>
+  <joint name="base_right_light_sensor_joint" type="fixed">
+    <origin xyz="0.0246 -0.1580 0.042" rpy="0 0 -1.0" />
+    <parent link="base_link" />
+    <child link="right_light_sensor_link" />
+  </joint>
+  <joint name="base_right_front_light_sensor_joint" type="fixed">
+    <origin xyz="0.0938 -0.1295 0.042" rpy="0 0 -0.9438" />
+    <parent link="base_link" />
+    <child link="right_front_light_sensor_link" />
+  </joint>
+  <joint name="base_right_center_light_sensor_joint" type="fixed">
+    <origin xyz="0.1425 -0.0727 0.042" rpy="0 0 -0.4719" />
+    <parent link="base_link" />
+    <child link="right_center_light_sensor_link" />
+  </joint>
+  <!-- Simulation sensors -->
+  <xacro:sim_create_light_sensors/>
 </robot>

File: create_description/urdf/create_2_gazebo.urdf.xacro (robot description, xacro)
@@ -1,3 +1,39 @@
 <?xml version="1.0" ?>
 <robot xmlns:xacro="http://ros.org/wiki/xacro">
+  <xacro:macro name="sim_create_light_sensor" params="prefix topic">
+    <gazebo reference="${prefix}_link">
+      <sensor type="ray" name="${prefix}">
+        <always_on>true</always_on>
+        <update_rate>20.0</update_rate>
+        <pose>0 0 0 0 0 0</pose>
+        <visualize>false</visualize>
+        <ray>
+          <scan>
+            <horizontal>
+              <samples>1</samples>
+              <resolution>1</resolution>
+              <min_angle>0</min_angle>
+              <max_angle>0</max_angle>
+            </horizontal>
+          </scan>
+          <range>
+            <min>0.0160</min>
+            <max>0.05</max>
+            <resolution>0.1</resolution>
+          </range>
+        </ray>
+        <plugin name="gazebo_${prefix}" filename="libcreate_light_sensor_plugin.so">
+          <topicName>${topic}</topicName>
+        </plugin>
+      </sensor>
+    </gazebo>
+  </xacro:macro>
+  <xacro:macro name="sim_create_light_sensors">
+    <xacro:sim_create_light_sensor prefix="left_light_sensor" topic="/sim/light_left" />
+    <xacro:sim_create_light_sensor prefix="left_front_light_sensor" topic="/sim/light_leftfront" />
+    <xacro:sim_create_light_sensor prefix="left_center_light_sensor" topic="/sim/light_leftcenter" />
+    <xacro:sim_create_light_sensor prefix="right_light_sensor" topic="/sim/light_right" />
+    <xacro:sim_create_light_sensor prefix="right_front_light_sensor" topic="/sim/light_rightfront" />
+    <xacro:sim_create_light_sensor prefix="right_center_light_sensor" topic="/sim/light_rightcenter" />
+  </xacro:macro>
 </robot>

Commit message: model fixes for gazebo

File: create_description/urdf/create_2.urdf.xacro (robot description, xacro)
@@ -3,6 +3,7 @@
   <xacro:include filename="$(find create_description)/urdf/create_base.urdf.xacro" />
   <xacro:include filename="$(find create_description)/urdf/create_2_gazebo.urdf.xacro" />
+  <xacro:property name="create_2_mesh" value="file://$(find create_description)/meshes/create_2.dae"/>
   <xacro:create_base wheel_separation="0.235" base_diameter="0.3485">
-    <mesh filename="package://create_description/meshes/create_2.dae" />
+    <mesh filename="${create_2_mesh}" />
   </xacro:create_base>
 </robot>

File: create_description/urdf/create_base.urdf.xacro (robot description, xacro)
@@ -31,29 +31,11 @@
   <xacro:macro name="create_base" params="diffdrive_update_rate:=40 wheel_separation wheel_radius:=0.036 wheel_width:=0.024 wheel_torque:=1.0 wheel_accel:=1.8 mass_kg:=3.5 base_diameter *mesh">
     <xacro:include filename="$(find create_description)/urdf/create_base_gazebo.urdf.xacro" />
-    <link name="base_footprint">
-    <inertial>
-      <origin xyz="0 0 0" />
-      <mass value="0.001" />
-      <inertia ixx="0.0001" ixy="0.0" ixz="0.0" iyy="0.0001" iyz="0.0" izz="0.0001" />
-    </inertial>
-    <visual>
-      <origin xyz="0 0 0" rpy="0 0 0" />
-      <geometry>
-        <box size="0.001 0.001 0.001" />
-      </geometry>
-      <material name="Green" />
-    </visual>
-    <collision>
-      <origin xyz="0 0 0.017" rpy="0 0 0" />
-      <geometry>
-        <box size="0.001 0.001 0.001" />
-      </geometry>
-    </collision>
-    </link>
+    <link name="base_footprint" />
     <link name="base_link">
     <inertial>
       <mass value="2" />
       <origin xyz="0 0 0.0" />
-      <inertia ixx="0.01" ixy="0.0" ixz="0.0" iyy="0.01" iyz="0.0" izz="0.5" />
+      <!-- <inertia ixx="0.01" ixy="0.0" ixz="0.0" iyy="0.01" iyz="0.0" izz="0.5" /> -->
+      <inertia ixx="0.02" ixy="0.0" ixz="0.0" iyy="0.02" iyz="0.0" izz="0.04" />
     </inertial>
     <visual>
@@ -70,5 +52,5 @@
     </collision>
     </link>
-    <link name="wall_sensor_link">
+    <!-- <link name="wall_sensor_link">
     <inertial>
       <mass value="0.01" />
@@ -104,5 +86,5 @@
       <inertia ixx="0.001" ixy="0.0" ixz="0.0" iyy="0.001" iyz="0.0" izz="0.001" />
     </inertial>
-    </link>
+    </link> -->
     <joint name="base_footprint_joint" type="fixed">
       <origin xyz="0 0 0.017" rpy="0 0 0" />
@@ -110,5 +92,5 @@
       <child link="base_link" />
     </joint>
-    <joint name="base_wall_sensor_joint" type="fixed">
+    <!-- <joint name="base_wall_sensor_joint" type="fixed">
       <origin xyz="0.09 -0.120 0.042" rpy="0 0 -1.0" />
       <parent link="base_link" />
@@ -134,5 +116,5 @@
       <parent link="base_link" />
       <child link="rightfront_cliff_sensor_link" />
-    </joint>
+    </joint> -->
     <xacro:create_wheel prefix="left" y_offset="${wheel_separation / 2}" wheel_radius="${wheel_radius}" wheel_width="${wheel_width}"/>
     <xacro:create_wheel prefix="right" y_offset="${wheel_separation / -2}" wheel_radius="${wheel_radius}" wheel_width="${wheel_width}"/>
@@ -204,7 +186,7 @@
     <!-- Simulation sensors -->
     <xacro:sim_create_base/>
-    <xacro:sim_create_wall_sensor/>
+    <!-- <xacro:sim_create_wall_sensor/>
     <xacro:sim_create_cliff_sensors/>
-    <xacro:sim_imu/>
+    <xacro:sim_imu/> -->
   </xacro:macro>
 </robot>
